File: Electronics/Project work/Electronics Circuit/Electronics Project.kicad_sch (KiCad schematic)
At the start: 0 parts

Commit message: quick save
Parts:
- added C1: 100n, symbol Device:C
- added C2: 1u, symbol Device:C
- added C3: 10u, 10u, symbol Device:C
- added D1: D, symbol Simulation_SPICE:D
- added R1: 12k, symbol Device:R
- added R2: 100k, symbol Device:R
- added R3: 50k, symbol Device:R
- added R4: 10k, symbol Device:R
- added R5: 11.7k, symbol Device:R
- added R6: 10k, 10k, symbol Device:R
- added U1, U2, U3, U4: ${SIM.PARAMS}, symbol Simulation_SPICE:OPAMP
- added V1: VPULSE, symbol Simulation_SPICE:VPULSE
- added V10, V2, V4, V6: 15, symbol Simulation_SPICE:VDC
- added V3, V5, V7, V9: -15, symbol Simulation_SPICE:VDC
- added V8: 5, symbol Simulation_SPICE:VDC
Connections:
- new net: U2.3 (V+), V4.1
- new net: C1.1, R1.2, R2.1, U1.2 (-)
- new net: U1.3 (V+), V2.1
- new net: U1.4 (V-), V3.1
- new net: C1.2, R2.2, U1.5, U2.1 (+)
- new net: R1.1, V1.1
- new net: U2.4 (V-), V5.1
- new net: R5.1, R6.2, U3.5
- new net: R4.2, R5.2, U3.2 (-)
- new net: U3.1 (+), V8.1
- new net: C2.1, D1.1 (K), R3.2, U2.2 (-), U4.1 (+)
- new net: C3.1, R6.1
- new net: U3.4 (V-), V7.1
- new net: U3.3 (V+), V6.1
- new net: R4.1, U4.2 (-), U4.5
- new net: D1.2 (A), U2.5
- new net: U4.4 (V-), V9.1
- new net: U4.3 (V+), V10.1
- new net 0: C2.2, C3.2, R3.1, U1.1 (+), V1.2, V10.2, V2.2, V3.2, V4.2, V5.2, V6.2, V7.2, V8.2, V9.2
Other:
- note added: "100Hz: PULSE(-5 5 0 1u 1u 5m 10m)"
- note added: "1kHz: Pulse(-5 5 0 1u 1u 0.5m 1m)"
- note added: "Final Output"
- note added: "Inverting Normalization (0.1V - 10V)"
- note added: "Low Pass Filter"
- note added: "Peak Detection"
- note added: "Triangle Wave Generation"
- note added: "Voltage Buffer"
